File: trackingDevice_circuitBoard/trackingDevice_circuitBoard.kicad_pcb (KiCad board)
At the start: 2 copper layers, 50.8 x 45.7 mm, 16 parts, among them P1 Digital, P4 Analog, Q1 Q_NPN_EBC, Q2 Q_NPN_EBC, Q3 Q_NPN_EBC, U1 HC-12, U2 GY-NEO6MV2, U3 TP4056

Commit message: Added veroboard/stripboard drill marks + corrected error in tracking device circuit
Parts:
- Q1: footprint TO_SOT_Packages_THT:TO-126_Vertical -> TO_SOT_Packages_THT:TO-92_Inline_Wide

Commit message: Modified resistor values to be more power-efficient
Parts:
- R1: value 1000R -> 10kR
- R2: value 2000R -> 47kR
- R3, R4, R5, R6: value 1000R -> 27kR
- R7: value 1000R -> 4.7kR
Changed lines of the file:
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@@
     (links 30)
     (no_connects 2)
-    (area 17.550001 19.844999 143.175 98.195001)
+    (area 30.429999 35.509999 81.330001 81.330001)
     (thickness 1.6)
     (drawings 102)
@@
   (title_block
     (title "Arduino GPS Tracker - Tracking Device")
-    (date 2018-08-09)
+    (date 2018-08-10)
     (rev 1)
     (company "By Megasaturnv")
@@
       (effects (font (size 1 1) (thickness 0.15)))
     )
-    (fp_text value 1000R (at 5.08 1.27 270) (layer F.Fab)
+    (fp_text value 10kR (at 5.08 1.27 270) (layer F.Fab)
       (effects (font (size 1 1) (thickness 0.15)))
     )
@@
       (effects (font (size 1 1) (thickness 0.15)))
     )
-    (fp_text value 2000R (at 5.08 -1.27 270) (layer F.Fab)
+    (fp_text value 47kR (at 5.08 -1.27 270) (layer F.Fab)
       (effects (font (size 1 1) (thickness 0.15)))
     )
@@
       (effects (font (size 1 1) (thickness 0.15)))
     )
-    (fp_text value 1000R (at 5.08 1.27) (layer F.Fab)
+    (fp_text value 27kR (at 5.08 1.27) (layer F.Fab)
       (effects (font (size 1 1) (thickness 0.15)))
     )
@@
       (effects (font (size 1 1) (thickness 0.15)))
     )
-    (fp_text value 1000R (at 5.08 -1.27 90) (layer F.Fab)
+    (fp_text value 27kR (at 5.08 -1.27 90) (layer F.Fab)
       (effects (font (size 1 1) (thickness 0.15)))
     )
@@
       (effects (font (size 1 1) (thickness 0.15)))
     )
-    (fp_text value 1000R (at 5.08 -1.27 180) (layer F.Fab)
+    (fp_text value 27kR (at 5.08 -1.27 180) (layer F.Fab)
       (effects (font (size 1 1) (thickness 0.15)))
     )
@@
       (effects (font (size 1 1) (thickness 0.15)))
     )
-    (fp_text value 1000R (at 5.08 -1.27 270) (layer F.Fab)
+    (fp_text value 27kR (at 5.08 -1.27 270) (layer F.Fab)
       (effects (font (size 1 1) (thickness 0.15)))
     )
@@
       (effects (font (size 1 1) (thickness 0.15)))
     )
-    (fp_text value 1000R (at 7.62 -1.27 90) (layer F.Fab)
-      (effects (font (size 1 1) (thickness 0.15)))
-    )
+    (fp_text value 4.7kR (at 7.62 -1.27 90) (layer F.Fab)
+      (effects (font (size 1 1) (thickness 0.15)))
+    )
